Commit message: added joy_teleop

File: src/rosoomba_description/urdf/gazebo_original.xacro (robot description, xacro)
@@ -90,4 +90,13 @@
           </range>
         </ray>
+        <plugin name="wall_sensor_plugin" filename="libgazebo_ros_range.so">
+          <ros>
+            <namespace></namespace>
+            <remapping>~/out:=wall_sensor/range</remapping>
+          </ros>
+          <output_type>sensor_msgs/Range</output_type>
+          <radiation_type>infrared</radiation_type>
+          <frame_name>wall_sensor_link</frame_name>
+        </plugin>
       </sensor>
     </gazebo>
@@ -115,4 +124,13 @@
           </range>
         </ray>
+        <plugin name="left_cliff_sensor_plugin" filename="libgazebo_ros_range.so">
+          <ros>
+            <namespace></namespace>
+            <remapping>~/out:=left_cliff_sensor/range</remapping>
+          </ros>
+          <output_type>sensor_msgs/Range</output_type>
+          <radiation_type>infrared</radiation_type>
+          <frame_name>left_cliff_sensor_link</frame_name>
+        </plugin>
       </sensor>
     </gazebo>
@@ -138,4 +156,13 @@
           </range>
         </ray>
+        <plugin name="right_cliff_sensor_plugin" filename="libgazebo_ros_range.so">
+          <ros>
+            <namespace></namespace>
+            <remapping>~/out:=right_cliff_sensor/range</remapping>
+          </ros>
+          <output_type>sensor_msgs/Range</output_type>
+          <radiation_type>infrared</radiation_type>
+          <frame_name>right_cliff_sensor_link</frame_name>
+        </plugin>
       </sensor>
     </gazebo>
@@ -161,4 +188,13 @@
           </range>
         </ray>
+        <plugin name="leftfront_cliff_sensor_plugin" filename="libgazebo_ros_range.so">
+          <ros>
+            <namespace></namespace>
+            <remapping>~/out:=leftfront_cliff_sensor/range</remapping>
+          </ros>
+          <output_type>sensor_msgs/Range</output_type>
+          <radiation_type>infrared</radiation_type>
+          <frame_name>leftfront_cliff_sensor_link</frame_name>
+        </plugin>
       </sensor>
     </gazebo>
@@ -184,4 +220,13 @@
           </range>
         </ray>
+        <plugin name="rightfront_cliff_sensor_plugin" filename="libgazebo_ros_range.so">
+          <ros>
+            <namespace></namespace>
+            <remapping>~/out:=rightfront_cliff_sensor/range</remapping>
+          </ros>
+          <output_type>sensor_msgs/Range</output_type>
+          <radiation_type>infrared</radiation_type>
+          <frame_name>rightfront_cliff_sensor_link</frame_name>
+        </plugin>
       </sensor>
     </gazebo>

File: src/rosoomba_description/urdf/rosoomba.urdf.xacro (robot description, xacro)
@@ -2,14 +2,10 @@
 <robot name="rosoomba" xmlns:xacro="http://ros.org/wiki/xacro">
   <xacro:property name="package_path" value="$(find rosoomba_description)" />
-  <xacro:include filename="${package_path}/urdf/params.urdf.xacro" />
-  <xacro:include filename="${package_path}/urdf/base.urdf.xacro" />
-  <xacro:include filename="${package_path}/urdf/wheel.urdf.xacro" />
+  <xacro:include filename="${package_path}/urdf/params.xacro" />
+  <xacro:include filename="${package_path}/urdf/rosoomba_core.xacro" />
+  <xacro:include filename="${package_path}/urdf/wheel.xacro" />
   <xacro:create_wheel prefix="left" y_offset="${wheel_separation / 2}" wheel_radius="${wheel_radius}" wheel_width="${wheel_width}"/>
   <xacro:create_wheel prefix="right" y_offset="${wheel_separation / -2}" wheel_radius="${wheel_radius}" wheel_width="${wheel_width}"/>
-  <!-- Gazebo simulation sensors -->
-  <xacro:include filename="${package_path}/urdf/gazebo.urdf.xacro" />
-  <xacro:sim_create_base/>
-  <xacro:sim_create_wall_sensor/>
-  <xacro:sim_create_cliff_sensors/>
-  <xacro:sim_imu/>
+  <!-- <xacro:include filename="${package_path}/urdf/gazebo_control.xacro" /> -->
+  <xacro:include filename="${package_path}/urdf/ros2_control.xacro" />
 </robot>

File: src/rosoomba_description/urdf/rosoomba_core.xacro (robot description, xacro)
@@ -2,9 +2,9 @@
 <robot xmlns:xacro="http://ros.org/wiki/xacro">
   <link name="base_footprint">
-    <inertial>
+    <!-- <inertial>
       <mass value="0.01" />
       <origin xyz="0 0 0" />
       <inertia ixx="0.00002083" ixy="0.0" ixz="0.0" iyy="0.00002083" iyz="0.0" izz="0.0000125" />
-    </inertial>
+    </inertial> -->
   </link>
   <link name="base_link">

File: src/rosoomba_description/urdf/wheel.xacro (robot description, xacro)
@@ -5,6 +5,6 @@
     <inertial>
       <origin xyz="0 0 0" />
-      <mass value="0.01" />
-      <inertia ixx="0.001" ixy="0.0" ixz="0.0" iyy="0.001" iyz="0.0" izz="0.001" />
+      <mass value="0.2" />
+      <inertia ixx="0.002" ixy="0.0" ixz="0.0" iyy="0.002" iyz="0.0" izz="0.002" />
     </inertial>
     <visual>
@@ -21,4 +21,13 @@
     </collision>
     </link>
+    <!-- Gazebo material properties for wheel friction -->
+    <gazebo reference="${prefix}_wheel_link">
+      <mu1>1.0</mu1>
+      <mu2>1.0</mu2>
+      <kp>1000000.0</kp>
+      <kd>100.0</kd>
+      <minDepth>0.001</minDepth>
+      <maxVel>1.0</maxVel>
+    </gazebo>
    <joint name="${prefix}_wheel_joint" type="continuous">
       <origin xyz="0 ${y_offset} 0.015" rpy="0 0 0" />
